File: hardware/MerlinESP.kicad_pcb (KiCad board)
At the start: 4 copper layers, 61.2 x 35 mm, 89 parts, among them J2 USB4105, J3 950066002000000, J5 UF.L, J6 950066002000000, J7 950066002000000, J8 950066002000000, K1 G6K-2F DC5, K2 G6K-2F DC5, Q1 2N7002KL3A-TP, Q3 40 MHz, Q4 2N7002KL3A-TP, SW1 5134TR, SW2 5134TR, U1 950066003500000, U2 TPS74633-Q1, U3 TSV991AIQ1T, U4 BGS12WN6E6327XTSA1, U5 LMR51610YFDBVR, U7 ESP32-C6

Commit message: Fixed pin 14 no adc issue
Connections:
- U7 pad 12: unconnected-(U7-MTCK-Pad12) -> /MCU/Light_Flashing
- U7 pad 14: /MCU/Light_Flashing -> unconnected-(U7-GPIO8-Pad14)
