File: hardware/mcu.kicad_sch (KiCad schematic)
At the start: 33 parts, among them J5 UF.L, Q3 40 MHz, SW1 5134TR, SW2 5134TR, U4 BGS12WN6E6327XTSA1, U7 ESP32-C6

Commit message: Fixed pin 14 no adc issue
Connections:
- net Light_Flashing: now also U7.12 (MTCK); no longer U7.14 (GPIO8)
Changed lines of the file:
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@@
 	(hierarchical_label "Light_Flashing"
 		(shape input)
-		(at 96.52 96.52 180)
+		(at 142.24 106.68 0)
 		(effects
 			(font
 				(size 1.27 1.27)
 			)
-			(justify right)
+			(justify left)
 		)
 	)
